Commit message: Implement working pick-and-place simulation for cooka robot
- Switch arm joints to velocity command interface with per-joint JTC PID
  (P=50, I=0, D=0.5) to eliminate oscillation caused by position_proportional_gain
- Add world→base_link fixed joint to anchor robot against reaction forces
- Set gravity=false on all arm links; restore spawner nodes for controller activation
- Implement full 10-step pnp_node state machine with FollowJointTrajectory action,
  two-phase SCARA extend (joint-space to SAFE_Y, then Cartesian IK sweep to target),
  and DetachableJoint-based payload attachment
- Spawn payload with gravity=false at (0.3, 0.5, 0.425) at t=5s; pnp_node sends
  detach on startup so payload stays free until gripper closes at pick A
- Home position: scara_j1=120°, scara_j2=-240°, wrist_z≈-120°
- Add live monitor node (joint pos/vel + FK EE position at 10 Hz)

Verified: robot stable, EE reaches pick A (0.3, 0.319, 0.525) and drop B
(1.6, 0.319, 1.1), payload attaches/detaches correctly via DetachableJoint.

Co-Authored-By: Claude Sonnet 4.6 <noreply@anthropic.com>

File: cooka_description/urdf/cooka.xacro (robot description, xacro)
@@ -7,4 +7,12 @@
   <xacro:include filename="$(find cooka_description)/urdf/cooka.gazebo" />
 </xacro:if>
+<!-- Fixes base_link to the Gazebo world frame so joint reaction forces
+     do not move the whole robot body. -->
+<link name="world"/>
+<joint name="world_joint" type="fixed">
+  <parent link="world"/>
+  <child link="base_link"/>
+  <origin xyz="0 0 0" rpy="0 0 0"/>
+</joint>
 <link name="base_link">
   <inertial>
